File: Hardware/Schematic.sch (EAGLE design)
At the start: 105 parts, among them IC1 BQ25180YBGR_BQ25180YBGR, IC3 BMA421, IC4 DRV2605YZFR, IC9 RT6160AWSC, J1 503480-2400, J2 TC2030-IDC, J4 KH-TYPE-C-16P, Q1 20V/4.2A/52mΩ/1.4W, Q3 SI1308EDL-T1-GE3, U1 NRF52840_QF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

Commit message: Final Project
Parts:
- C1-EP-DR: value 22uF -> 10uF
- C10: value 820pF -> N.C.
- C11: value 820pF -> 100pF
- C2-EP-DR: value 22uF -> 4.7uF/25V
- renumbered C1-EP-DR1 to C2-EP-DR, C9\1 to C11, C9\2 to C10
Connections:
- removed net SDA/1.4C: IC4.SDA
- net SDA: now also IC4.SDA
Other:
- note added: "18.04.2026 11:25"
- note added: "E-Paper &Peripherals"
- note added: "InkTime v6"
- note added: "MCU, Power, IMU, SWD"
- note added: "drawn by: Balica Andrei-Sebastian"
Changed lines of the file:
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@@
 <part name="GND24" library="InkTime_v5" deviceset="HECTOR_WATCH_2_GND" device="" value="GND"/>
 <part name="GND25" library="InkTime_v5" deviceset="HECTOR_WATCH_2_GND" device="" value="GND"/>
-<part name="C9\1" library="InkTime_v5" deviceset="NORDIC_NRF_3_CAPACITOR" device="_0201_L" value="820pF"/>
-<part name="C9\2" library="InkTime_v5" deviceset="NORDIC_NRF_3_CAPACITOR" device="_0201_L" value="820pF"/>
+<part name="C11" library="InkTime_v5" deviceset="NORDIC_NRF_3_CAPACITOR" device="_0201_L" value="100pF"/>
+<part name="C10" library="InkTime_v5" deviceset="NORDIC_NRF_3_CAPACITOR" device="_0201_L" value="N.C."/>
 <part name="L1" library="InkTime_v5" deviceset="MLP2016SR47MT0S1_FTC252012SR47MBCA" device="" value="3.9nH"/>
 <part name="C3" library="InkTime_v5" deviceset="NORDIC_NRF_3_CAPACITOR" device="_0201_L" value="1pF"/>
@@
 <part name="FRAME2" library="InkTime_v5" deviceset="FRAMES_A3L-LOC" device=""/>
 <part name="SJ1" library="InkTime_v5" deviceset="ESP32_C6_LIBRARY_7_JUMPER_SJ" device=""/>
-<part name="C1-EP-DR" library="InkTime_v5" deviceset="NORDIC_NRF_3_CAPACITOR" device="_0201_L" value="22uF"/>
+<part name="C1-EP-DR" library="InkTime_v5" deviceset="NORDIC_NRF_3_CAPACITOR" device="_0201_L" value="10uF"/>
 <part name="GND34" library="InkTime_v5" deviceset="HECTOR_WATCH_2_GND" device="" value="GND"/>
 <part name="D2" library="InkTime_v5" deviceset="ESP32_C6_LIBRARY_5_MBR0530" device="" value="MBR0530"/>
 <part name="L5" library="InkTime_v5" deviceset="ESP32_C6_LIBRARY_2_744043680" device="IND_4828-WE-TPC_WRE" value="68uH"/>
-<part name="C1-EP-DR1" library="InkTime_v5" deviceset="NORDIC_NRF_3_CAPACITOR" device="_0201_L" value="22uF"/>
+<part name="C2-EP-DR" library="InkTime_v5" deviceset="NORDIC_NRF_3_CAPACITOR" device="_0201_L" value="4.7uF/25V"/>
 <part name="D5" library="InkTime_v5" deviceset="ESP32_C6_LIBRARY_5_MBR0530" device="" value="MBR0530"/>
 <part name="D4" library="InkTime_v5" deviceset="ESP32_C6_LIBRARY_5_MBR0530" device="" value="MBR0530"/>
@@
 <text x="175.26" y="-365.76" size="3.81" layer="97" font="custom">USB C Connector &amp; ESD
 Protection</text>
+<text x="269.24" y="-421.64" size="3.81" layer="94" align="top-center">E-Paper &amp;Peripherals</text>
+<text x="297.18" y="-419.1" size="1.778" layer="94">drawn by: Balica Andrei-Sebastian</text>
+<text x="297.18" y="-424.18" size="1.778" layer="94">InkTime v6</text>
+<text x="297.18" y="-429.26" size="1.778" layer="94">18.04.2026 11:25</text>
+<text x="297.18" y="-137.16" size="1.778" layer="94">drawn by: Balica Andrei-Sebastian</text>
+<text x="297.18" y="-142.24" size="1.778" layer="94">InkTime v6</text>
+<text x="297.18" y="-147.32" size="1.778" layer="94">18.04.2026 11:25</text>
+<text x="269.24" y="-137.16" size="3.81" layer="94" align="top-center">MCU, Power,
+IMU, SWD</text>
 </plain>
 <instances>
@@
 <attribute name="VALUE" x="243.84" y="2.54" size="1.778" layer="96"/>
 </instance>
-<instance part="C9\1" gate="C$1" x="233.68" y="15.24" smashed="yes">
+<instance part="C11" gate="C$1" x="233.68" y="15.24" smashed="yes">
 <attribute name="NAME" x="235.204" y="15.621" size="1.778" layer="95"/>
 <attribute name="VALUE" x="235.204" y="10.541" size="1.778" layer="96"/>
 </instance>
-<instance part="C9\2" gate="C$1" x="246.38" y="15.24" smashed="yes">
+<instance part="C10" gate="C$1" x="246.38" y="15.24" smashed="yes">
 <attribute name="NAME" x="247.904" y="15.621" size="1.778" layer="95"/>
 <attribute name="VALUE" x="247.904" y="10.541" size="1.778" layer="96"/>
@@
 </instance>
 <instance part="FRAME1" gate="G$1" x="-45.72" y="-157.48" smashed="yes">
-<attribute name="DRAWING_NAME" x="298.45" y="-142.24" size="2.54" layer="94"/>
-<attribute name="LAST_DATE_TIME" x="298.45" y="-147.32" size="2.286" layer="94"/>
 <attribute name="SHEET" x="311.785" y="-152.4" size="2.54" layer="94"/>
 </instance>
 <instance part="FRAME2" gate="G$1" x="-45.72" y="-439.42" smashed="yes">
-<attribute name="DRAWING_NAME" x="298.45" y="-424.18" size="2.54" layer="94"/>
-<attribute name="LAST_DATE_TIME" x="298.45" y="-429.26" size="2.286" layer="94"/>
 <attribute name="SHEET" x="311.785" y="-434.34" size="2.54" layer="94"/>
 </instance>
@@
 <attribute name="NAME" x="-11.0698" y="-230.3399" size="3.48" layer="95" ratio="10"/>
 </instance>
-<instance part="C1-EP-DR1" gate="C$1" x="10.16" y="-241.3" smashed="yes">
+<instance part="C2-EP-DR" gate="C$1" x="10.16" y="-241.3" smashed="yes">
 <attribute name="NAME" x="11.684" y="-240.919" size="1.778" layer="95"/>
 <attribute name="VALUE" x="11.684" y="-245.999" size="1.778" layer="96"/>
@@
 </segment>
 <segment>
-<pinref part="C9\2" gate="C$1" pin="2"/>
+<pinref part="C10" gate="C$1" pin="2"/>
 <wire x1="246.38" y1="10.16" x2="246.38" y2="7.62" width="0.1524" layer="91"/>
 <pinref part="GND25" gate="1" pin="GND"/>
 </segment>
 <segment>
-<pinref part="C9\1" gate="C$1" pin="2"/>
+<pinref part="C11" gate="C$1" pin="2"/>
 <wire x1="233.68" y1="10.16" x2="233.68" y2="7.62" width="0.1524" layer="91"/>
 <pinref part="GND24" gate="1" pin="GND"/>
@@
 <wire x1="254" y1="20.32" x2="246.38" y2="20.32" width="0.1524" layer="91"/>
 <wire x1="246.38" y1="20.32" x2="246.38" y2="17.78" width="0.1524" layer="91"/>
-<pinref part="C9\2" gate="C$1" pin="1"/>
+<pinref part="C10" gate="C$1" pin="1"/>
 <wire x1="254" y1="20.32" x2="254" y2="66.04" width="0.1524" layer="91"/>
 <junction x="254" y="20.32"/>
@@
 <wire x1="241.3" y1="20.32" x2="233.68" y2="20.32" width="0.1524" layer="91"/>
 <wire x1="233.68" y1="20.32" x2="233.68" y2="17.78" width="0.1524" layer="91"/>
-<pinref part="C9\1" gate="C$1" pin="1"/>
+<pinref part="C11" gate="C$1" pin="1"/>
 <label x="233.68" y="20.32" size="1.778" layer="95"/>
 </segment>
@@
 <junction x="10.16" y="-248.92"/>
 <wire x1="10.16" y1="-248.92" x2="10.16" y2="-246.38" width="0.1524" layer="91"/>
-<pinref part="C1-EP-DR1" gate="C$1" pin="2"/>
+<pinref part="C2-EP-DR" gate="C$1" pin="2"/>
 <wire x1="5.08" y1="-233.68" x2="5.08" y2="-203.2" width="0.1524" layer="91"/>
 <junction x="5.08" y="-233.68"/>
@@
 <net name="N$15" class="0">
 <segment>
-<pinref part="C1-EP-DR1" gate="C$1" pin="1"/>
+<pinref part="C2-EP-DR" gate="C$1" pin="1"/>
 <wire x1="10.16" y1="-238.76" x2="10.16" y2="-236.22" width="0.1524" layer="91"/>
 <wire x1="10.16" y1="-236.22" x2="15.24" y2="-236.22" width="0.1524" layer="91"/>
@@
 </segment>
 </net>
-<net name="SDA/1.4C" class="0">
-<segment>
-<pinref part="IC4" gate="G$1" pin="SDA"/>
-<wire x1="256.54" y1="-220.98" x2="238.76" y2="-220.98" width="0.1524" layer="91"/>
-<label x="238.76" y="-220.98" size="1.778" layer="95" font="custom" rot="R180" xref="yes"/>
-</segment>
-</net>
 <net name="OUT-" class="0">
 <segment>
@@
 <label x="139.7" y="-20.32" size="1.778" layer="95" rot="R180" xref="yes"/>
 </segment>
-</net>
+<segment>
+<pinref part="IC4" gate="G$1" pin="SDA"/>
+<wire x1="256.54" y1="-220.98" x2="238.76" y2="-220.98" width="0.1524" layer="91"/>
+<label x="238.76" y="-220.98" size="1.778" layer="95" font="custom" rot="R180" xref="yes"/>
+</segment>
+</net>
